Commit message: added mesh files

File: nodes/bot.urdf (robot description, URDF)
Before this commit: robot basics, 1 links, 0 joints
Links:
- link base_link: geometry visual mesh filename=package://ros_learning/meshes/wheel.dae

Commit message: Improvement

File: nodes/bot.urdf (robot description, URDF)
Before this commit: robot basics, 1 links, 0 joints
Links:
- link base_link: geometry visual mesh filename=package://ros_learning/meshes/body.stl
