Commit message: added tool frame

File: urdf/scara.urdf (robot description, URDF)
Before this commit: robot scara, 4 links, 3 joints
Links:
- added link tool
Joints:
- added joint tool_to_link3: type fixed, parent link_3, child tool, origin xyz=0 0 -0.175
- joint link1_to_base: origin xyz=1.15 0 3.01 -> xyz=0.100 0 0.301
- joint link2_to_link1: limit lower=-2.43 upper=2.43 effort=300 velocity=0.1 -> lower=-2.70 upper=2.70 effort=300 velocity=0.1; origin xyz=2.25 0 1.025 -> xyz=0.225 0 0.100
- joint link3_to_link2: limit lower=-2.30 upper=0 effort=300 velocity=0.1 -> lower=-0.225 upper=0 effort=300 velocity=0.1; origin xyz=2.25 0 0 -> xyz=0.225 0 0

Commit message: IK

File: urdf/scara.urdf (robot description, URDF)
Before this commit: robot scara, 5 links, 4 joints
Links:
- added link end
Joints:
- removed joint link1_to_base
- removed joint link2_to_link1
- removed joint link3_to_link2
- added joint joint1: type revolute, parent base_link, child link_1, origin xyz=0.100 0 0.301, axis 0 0 1, limit lower=-2.70 upper=2.70 effort=300 velocity=0.1
- added joint joint2: type revolute, parent link_1, child link_2, origin xyz=0.225 0 0.100, axis 0 0 1, limit lower=-2.70 upper=2.70 effort=300 velocity=0.1
- added joint joint3: type prismatic, parent link_2, child link_3, origin xyz=0.225 0 0, axis 0 0 1, limit lower=-0.225 upper=0 effort=300 velocity=0.1
- added joint joint4: type revolute, parent link_3, child end, origin xyz=0 0 -0.175, axis 0 0 1, limit lower=-4.71 upper=4.71 effort=300 velocity=0.1
- joint tool_to_link3: origin xyz=0 0 -0.175 -> xyz=0 0 0; parent link_3 -> end

Commit message: ik improvement 2

File: urdf/scara.urdf (robot description, URDF)
Before this commit: robot scara, 6 links, 5 joints
Joints:
- joint joint1: limit lower=-2.70 upper=2.70 effort=300 velocity=0.1 -> lower=-1.57 upper=1.57 effort=300 velocity=0.1; origin xyz=0.100 0 0.301 -> xyz=0 0 0.301
- joint joint2: limit lower=-2.70 upper=2.70 effort=300 velocity=0.1 -> lower=-1 upper=1 effort=300 velocity=0.1
- joint joint3: limit lower=-0.225 upper=0 effort=300 velocity=0.1 -> lower=-0.205 upper=0 effort=300 velocity=0.1
- joint joint4: origin xyz=0 0 -0.175 -> xyz=0 0 -0.194
