Commit message: ik

File: urdf/robot_arm_6.urdf (robot description, URDF)
Before this commit: robot 6_axis_arm, 8 links, 7 joints
Joints:
- joint joint_1: limit lower=-2.96706 upper=2.96706 effort=1 velocity=3.92699081698724 -> lower=-1.57 upper=1.57 effort=300 velocity=0.1
- joint joint_2: limit lower=-2.094395 upper=2.094395 effort=1 velocity=2.61799387799149 -> lower=-1.57 upper=1.57 effort=300 velocity=0.1
- joint joint_3: limit lower=-2.181662 upper=2.70526 effort=1 velocity=2.85832571599111 -> lower=-1 upper=1 effort=300 velocity=0.1
- joint joint_4: limit lower=-4.712389 upper=4.712389 effort=1 velocity=3.92699081698724 -> lower=-1.57 upper=1.57 effort=300 velocity=0.1; origin xyz=0.010000 0.000000 0.164500 rpy=0.000000 0.000000 0.000000 -> xyz=-0.010000 0.000000 0.164500 rpy=0.000000 0.000000 0.000000
- joint joint_5: limit lower=-2.094395 upper=2.094395 effort=1 velocity=3.02168853397778 -> lower=-1.57 upper=1.57 effort=300 velocity=0.1
- joint joint_6: limit lower=-6.283185 upper=6.283185 effort=1 velocity=6.28318530717959 -> lower=-1.57 upper=1.57 effort=300 velocity=0.1
